File: KiCad/Projects/AtInverter_v2/_autosave-AtInverter_v2.kicad_pcb (KiCad board)
At the start: 2 copper layers, 83.8 x 94.6 mm, 116 parts, among them Q1 IRFB4020PBF, Q2 IRFB4020PBF, Q3 IRFB4020PBF, Q4 IRFB4020PBF, T1 ZMPT101B, U1 LM358N, U10 TLV61046ADB, U11 R-78HE5.0-0.3, U2 74LVC1G32, U3 LM393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

Commit message: ZMPT101B lib fix
Routing:
- net /!RESET: track 35.0 -> 33.6 mm
Changed lines of the file:
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@@
-	)
-	(segment
-		(start 69.596 118.8212)
-		(end 68.58 117.8052)
-		(width 0.15)
-		(layer "F.Cu")
-		(net 8)
 	)
 	(segment
