File: KiCad/Projects/AtInverter_v2/AtInverter_v2.kicad_pcb (KiCad board)
At the start: 2 copper layers, 83.8 x 94.6 mm, 116 parts, among them Q1 IRFB4020PBF, Q2 IRFB4020PBF, Q3 IRFB4020PBF, Q4 IRFB4020PBF, T1 ZMPT101B, U1 LM358N, U10 TLV61046ADB, U11 R-78HE5.0-0.3, U2 74LVC1G32, U3 LM393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

Commit message: Completed Overvoltage and Reset Protection Hardware Section
Parts:
- Rs1: value 100Ω -> 6.8Ω
- U2: value 74LVC1G32 -> SN74LVC1G32DBVR
Changed lines of the file:
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@@
 			)
 		)
-		(property "Value" "74LVC1G32"
+		(property "Value" "SN74LVC1G32DBVR"
 			(at 0 0 0)
 			(unlocked yes)
@@
 			)
 		)
-		(property "Value" "100Ω"
+		(property "Value" "6.8Ω"
 			(at 0 1.82 0)
 			(layer "F.Fab")
@@
 		)
 		(fp_text user "DTR"
-			(at 3.048 12.7 270)
+			(at 3.048 12.7 -90)
 			(unlocked yes)
 			(layer "F.SilkS")
